Commit message: new robot with right specifications

File: simulation_ws/src/ag2/urdf/ag2.xacro (robot description, xacro)
@@ -12,7 +12,8 @@
       <inertia ixx="0.0395416666667" ixy="0" ixz="0" iyy="0.106208333333" iyz="0" izz="0.106208333333"/>
     </inertial>
+    <!-- body -->
     <collision name="collision_chassis">
       <geometry>
-        <box size="0.5 0.3 0.07"/>
+        <cylinder radius="0.1" length="0.07"/>
       </geometry>
     </collision>
@@ -20,5 +21,5 @@
       <origin rpy="0 0 0" xyz="0 0 0"/>
       <geometry>
-        <box size="0.5 0.3 0.07"/>
+        <cylinder radius="0.1" length="0.07"/>
       </geometry>
       <material name="blue"/>
@@ -28,5 +29,5 @@
       <origin rpy=" 0 0 0" xyz="0.35 0 -0.05"/>
       <geometry>
-        <sphere radius="0.05"/>
+        <sphere radius="0.025"/>
       </geometry>
       <surface>
@@ -42,16 +43,20 @@
     </collision>
     <visual name="caster_front_visual">
-      <origin rpy=" 0 0 0" xyz="0.2 0 -0.05"/>
+      <origin rpy=" 0 0 0" xyz="0.075 0 -0.025"/>
       <geometry>
-        <sphere radius="0.05"/>
+        <sphere radius="0.025"/>
       </geometry>
     </visual>
-    </link>
+  </link>
   <link name="sensor_laser">
-    <xacro:cylinder_inertia mass="1" r="0.05" l="0.1" />
+    <inertial>
+      <origin xyz="0 0 0" rpy="0 0 0" />
+      <mass value="1" />
+      <xacro:cylinder_inertia mass="1" r="0.05" l="0.1" />
+    </inertial>
     <visual>
       <origin xyz="0 0 0" rpy="0 0 0" />
       <geometry>
-        <cylinder radius="0.05" length="0.1"/>
+        <cylinder radius="0.05" length="0.05"/>
       </geometry>
       <material name="white" />
@@ -60,10 +65,10 @@
       <origin xyz="0 0 0" rpy="0 0 0"/>
       <geometry>
-        <cylinder radius="0.05" length="0.1"/>
+        <cylinder radius="0.025" length="0.05"/>
       </geometry>
     </collision>
   </link>
   <joint name="joint_sensor_laser" type="fixed">
-    <origin xyz="0.15 0 0.05" rpy="0 0 0"/>
+    <origin xyz="0.05 0 0.05" rpy="0 0 0"/>
     <parent link="link_chassis"/>
     <child link="sensor_laser"/>
@@ -72,8 +77,8 @@
   <xacro:link_wheel name="link_right_wheel" />
   <!--   Joint for right wheel  -->
-  <xacro:joint_wheel name="joint_right_wheel"  child="link_right_wheel"  origin_xyz="-0.05 0.15 0"  />
+  <xacro:joint_wheel name="joint_right_wheel" child="link_right_wheel" origin_xyz="-0.02 0.125 0" />
   <!-- Left Wheel link -->
   <xacro:link_wheel name="link_left_wheel" />
   <!--   Joint for left wheel  -->
-  <xacro:joint_wheel name="joint_left_wheel"   child="link_left_wheel"   origin_xyz="-0.05 -0.15 0"  />
+  <xacro:joint_wheel name="joint_left_wheel" child="link_left_wheel" origin_xyz="-0.02 -0.125 0" />
 </robot>

Commit message: Robo finalizado

File: simulation_ws/src/ag2/urdf/ag2.xacro (robot description, xacro)
@@ -48,4 +48,27 @@
       </geometry>
     </visual>
+    <!-- caster back -->
+    <collision name="caster_back_collision">
+      <origin rpy=" 0 0 0" xyz="-0.35 0 -0.05"/>
+      <geometry>
+        <sphere radius="0.025"/>
+      </geometry>
+      <surface>
+        <friction>
+          <ode>
+            <mu>0</mu>
+            <mu2>0</mu2>
+            <slip1>1.0</slip1>
+            <slip2>1.0</slip2>
+          </ode>
+        </friction>
+      </surface>
+    </collision>
+    <visual name="caster_back_visual">
+      <origin rpy=" 0 0 0" xyz="-0.075 0 -0.025"/>
+      <geometry>
+        <sphere radius="0.025"/>
+      </geometry>
+    </visual>
   </link>
   <link name="sensor_laser">
